File: board/pod_27C512/pod_27C512.sch (KiCad schematic (older format))
At the start: 5 parts, among them J1 EXT_D, J2 EXT_ADDR, J3 VCC_Probe, J4 GND_Probe

Commit message: Update first pod schematics
Parts:
- added C1: 100nF, Capacitor_SMD:C_1206_3216Metric, symbol Device:C_Small
- added J5: ROM Lines, symbol Connector_Generic:Conn_02x14_Odd_Even
- added JP2, JP3, JP4, JP5, JP6: NO, Connector_PinHeader_2.54mm:PinHeader_1x02_P2.54mm_Vertical, symbol Device:Jumper_NO_Small
- added R1: 4.7K, Resistor_SMD:R_1206_3216Metric, symbol Device:R_Small
- added RN1: 10k, Resistor_THT:R_Array_SIP9, symbol Device:R_Network08
- added U1: 74HCT02, Package_SO:SO-14_3.9x8.65mm_P1.27mm, symbol 74xx:7400
Connections:
- net labels added: EXT_VCC, ~DIR_CE, ~SAFE_CE
- net labels removed: ~DIR_OE, ~SAFE_OE
- wire segments 138 -> 210
- no-connect marks 0 -> 1

Commit message: Update pod project
Parts:
- added D1: RED, LED_SMD:LED_1206_3216Metric, symbol Device:LED_Small
- added D2: GREEN, LED_SMD:LED_1206_3216Metric, symbol Device:LED_Small
- added R2: 1k, Resistor_SMD:R_1206_3216Metric, symbol Device:R_Small
- added R3: 470, Resistor_SMD:R_1206_3216Metric, symbol Device:R_Small
- J1, J2: footprint Connector_IDC:IDC-Header_2x20_P2.54mm_Vertical -> Connector_PinHeader_2.54mm:PinHeader_2x20_P2.54mm_Vertical
- J5: footprint (none) -> Connector_PinHeader_2.54mm:PinHeader_2x14_P2.54mm_Vertical
Connections:
- wire segments 210 -> 217
Changed lines of the file:
@@
 F 0 "J1" H 10200 3767 50  0000 C CNN
 F 1 "EXT_D" H 10200 3676 50  0000 C CNN
-F 2 "Connector_IDC:IDC-Header_2x20_P2.54mm_Vertical" H 10150 2650 50  0001 C CNN
+F 2 "Connector_PinHeader_2.54mm:PinHeader_2x20_P2.54mm_Vertical" H 10150 2650 50  0001 C CNN
 F 3 "~" H 10150 2650 50  0001 C CNN
 	1    10150 2650
@@
 F 0 "J2" H 10200 6117 50  0000 C CNN
 F 1 "EXT_ADDR" H 10200 6026 50  0000 C CNN
-F 2 "Connector_IDC:IDC-Header_2x20_P2.54mm_Vertical" H 10150 5000 50  0001 C CNN
+F 2 "Connector_PinHeader_2.54mm:PinHeader_2x20_P2.54mm_Vertical" H 10150 5000 50  0001 C CNN
 F 3 "~" H 10150 5000 50  0001 C CNN
 	1    10150 5000
@@
 Connection ~ 10550 5900
 $Comp
-L power:VCC #PWR?
+L power:VCC #PWR0101
 U 1 1 5FB7F9CB
 P 9850 6100
-F 0 "#PWR?" H 9850 5950 50  0001 C CNN
+F 0 "#PWR0101" H 9850 5950 50  0001 C CNN
 F 1 "VCC" H 9865 6273 50  0000 C CNN
 F 2 "" H 9850 6100 50  0001 C CNN
@@
 	9850 6000 9850 6100
 $Comp
-L power:VCC #PWR?
+L power:VCC #PWR0102
 U 1 1 5FB8884D
 P 9850 3750
-F 0 "#PWR?" H 9850 3600 50  0001 C CNN
+F 0 "#PWR0102" H 9850 3600 50  0001 C CNN
 F 1 "VCC" H 9865 3923 50  0000 C CNN
 F 2 "" H 9850 3750 50  0001 C CNN
@@
 	9050 2900 8900 2900
 $Comp
-L power:VCC #PWR?
+L power:VCC #PWR0103
 U 1 1 5FC724AB
 P 9150 2900
-F 0 "#PWR?" H 9150 2750 50  0001 C CNN
+F 0 "#PWR0103" H 9150 2750 50  0001 C CNN
 F 1 "VCC" H 9165 3073 50  0000 C CNN
 F 2 "" H 9150 2900 50  0001 C CNN
@@
 	9050 2850 9050 2900
 $Comp
-L power:GND #PWR?
+L power:GND #PWR0104
 U 1 1 5FC77E60
 P 10550 3800
-F 0 "#PWR?" H 10550 3550 50  0001 C CNN
+F 0 "#PWR0104" H 10550 3550 50  0001 C CNN
 F 1 "GND" H 10555 3627 50  0000 C CNN
 F 2 "" H 10550 3800 50  0001 C CNN
@@
 Connection ~ 10550 3650
 $Comp
-L power:GND #PWR?
+L power:GND #PWR0105
 U 1 1 5FC7D275
 P 10550 6100
-F 0 "#PWR?" H 10550 5850 50  0001 C CNN
+F 0 "#PWR0105" H 10550 5850 50  0001 C CNN
 F 1 "GND" H 10555 5927 50  0000 C CNN
 F 2 "" H 10550 6100 50  0001 C CNN
@@
 	9050 3350 9050 3400
 $Comp
-L power:GND #PWR?
+L power:GND #PWR0106
 U 1 1 5FC93A15
 P 9150 3400
-F 0 "#PWR?" H 9150 3150 50  0001 C CNN
+F 0 "#PWR0106" H 9150 3150 50  0001 C CNN
 F 1 "GND" H 9155 3227 50  0000 C CNN
 F 2 "" H 9150 3400 50  0001 C CNN
@@
 $EndComp
 $Comp
-L power:GND #PWR?
+L power:GND #PWR0107
 U 1 1 5FCFA381
 P 8900 2250
-F 0 "#PWR?" H 8900 2000 50  0001 C CNN
+F 0 "#PWR0107" H 8900 2000 50  0001 C CNN
 F 1 "GND" H 8905 2077 50  0000 C CNN
 F 2 "" H 8900 2250 50  0001 C CNN
@@
 	8900 2150 8900 2250
 $Comp
-L power:VCC #PWR?
+L power:VCC #PWR0108
 U 1 1 5FD01C5F
 P 8900 1000
-F 0 "#PWR?" H 8900 850 50  0001 C CNN
+F 0 "#PWR0108" H 8900 850 50  0001 C CNN
 F 1 "VCC" V 8915 1128 50  0000 L CNN
 F 2 "" H 8900 1000 50  0001 C CNN
@@
 	5150 1350 4750 1350
 $Comp
-L power:GND #PWR?
+L power:GND #PWR0109
 U 1 1 5FDA6912
 P 4800 1650
-F 0 "#PWR?" H 4800 1400 50  0001 C CNN
+F 0 "#PWR0109" H 4800 1400 50  0001 C CNN
 F 1 "GND" V 4805 1522 50  0000 R CNN
 F 2 "" H 4800 1650 50  0001 C CNN
@@
 	5250 2200 5400 2200
 $Comp
-L power:GND #PWR?
+L power:GND #PWR0110
 U 1 1 5FE0E8B3
 P 5150 2100
-F 0 "#PWR?" H 5150 1850 50  0001 C CNN
+F 0 "#PWR0110" H 5150 1850 50  0001 C CNN
 F 1 "GND" V 5155 1972 50  0000 R CNN
 F 2 "" H 5150 2100 50  0001 C CNN
@@
 $EndComp
 $Comp
-L power:GND #PWR?
+L power:GND #PWR0111
 U 1 1 5FE2D454
 P 6750 2100
-F 0 "#PWR?" H 6750 1850 50  0001 C CNN
+F 0 "#PWR0111" H 6750 1850 50  0001 C CNN
 F 1 "GND" V 6755 1972 50  0000 R CNN
 F 2 "" H 6750 2100 50  0001 C CNN
@@
 	6750 2100 6850 2100
 $Comp
-L power:VCC #PWR?
+L power:VCC #PWR0112
 U 1 1 5FE3C261
 P 7200 2100
-F 0 "#PWR?" H 7200 1950 50  0001 C CNN
+F 0 "#PWR0112" H 7200 1950 50  0001 C CNN
 F 1 "VCC" V 7215 2228 50  0000 L CNN
 F 2 "" H 7200 2100 50  0001 C CNN
@@
 F 0 "J5" H 6550 4517 50  0000 C CNN
 F 1 "ROM Lines" H 6550 4426 50  0000 C CNN
-F 2 "" H 6500 3700 50  0001 C CNN
+F 2 "Connector_PinHeader_2.54mm:PinHeader_2x14_P2.54mm_Vertical" H 6500 3700 50  0001 C CNN
 F 3 "~" H 6500 3700 50  0001 C CNN
 	1    6500 3700
@@
 	6300 4400 5800 4400
 $Comp
-L power:GND #PWR?
+L power:GND #PWR0113
 U 1 1 5FFADC5E
 P 5800 4500
-F 0 "#PWR?" H 5800 4250 50  0001 C CNN
+F 0 "#PWR0113" H 5800 4250 50  0001 C CNN
 F 1 "GND" H 5805 4327 50  0000 C CNN
 F 2 "" H 5800 4500 50  0001 C CNN
@@
 $EndComp
 $Comp
-L power:GND #PWR?
+L power:GND #PWR0114
 U 1 1 5FFE02FE
 P 1000 2100
-F 0 "#PWR?" H 1000 1850 50  0001 C CNN
+F 0 "#PWR0114" H 1000 1850 50  0001 C CNN
 F 1 "GND" H 1005 1927 50  0000 C CNN
 F 2 "" H 1000 2100 50  0001 C CNN
@@
 Text Label 2550 1400 2    50   ~ 0
 A11
+$Comp
+L Device:LED_Small D1
+U 1 1 601944B8
+P 1550 2550
+F 0 "D1" H 1550 2785 50  0000 C CNN
+F 1 "RED" H 1550 2694 50  0000 C CNN
+F 2 "LED_SMD:LED_1206_3216Metric" V 1550 2550 50  0001 C CNN
+F 3 "~" V 1550 2550 50  0001 C CNN
+	1    1550 2550
+	1    0    0    -1
+$EndComp
+$Comp
+L Device:R_Small R2
+U 1 1 6019F326
+P 1850 2550
+F 0 "R2" V 2046 2550 50  0000 C CNN
+F 1 "1k" V 1955 2550 50  0000 C CNN
+F 2 "Resistor_SMD:R_1206_3216Metric" H 1850 2550 50  0001 C CNN
+F 3 "~" H 1850 2550 50  0001 C CNN
+	1    1850 2550
+	0    -1   -1   0
+$EndComp
+Wire Wire Line
+	1750 2550 1650 2550
+$Comp
+L power:GND #PWR0115
+U 1 1 601B232D
+P 1350 2600
+F 0 "#PWR0115" H 1350 2350 50  0001 C CNN
+F 1 "GND" H 1355 2427 50  0000 C CNN
+F 2 "" H 1350 2600 50  0001 C CNN
+F 3 "" H 1350 2600 50  0001 C CNN
+	1    1350 2600
+	1    0    0    -1
+$EndComp
+Wire Wire Line
+	1450 2550 1350 2550
+Wire Wire Line
+	1350 2550 1350 2600
+Wire Wire Line
+	1950 2550 2400 2550
+Text Label 2400 2550 2    50   ~ 0
+EXT_VCC
+$Comp
+L Device:LED_Small D2
+U 1 1 601DEA89
+P 1550 3000
+F 0 "D2" H 1550 3235 50  0000 C CNN
+F 1 "GREEN" H 1550 3144 50  0000 C CNN
+F 2 "LED_SMD:LED_1206_3216Metric" V 1550 3000 50  0001 C CNN
+F 3 "~" V 1550 3000 50  0001 C CNN
+	1    1550 3000
+	1    0    0    -1
+$EndComp
+$Comp
+L Device:R_Small R3
+U 1 1 601DEF89
+P 1850 3000
+F 0 "R3" V 2046 3000 50  0000 C CNN
+F 1 "470" V 1955 3000 50  0000 C CNN
+F 2 "Resistor_SMD:R_1206_3216Metric" H 1850 3000 50  0001 C CNN
+F 3 "~" H 1850 3000 50  0001 C CNN
+	1    1850 3000
+	0    -1   -1   0
+$EndComp
+Wire Wire Line
+	1750 3000 1650 3000
+Wire Wire Line
+	1450 3000 950  3000
+Text Label 950  3000 0    50   ~ 0
+~SAFE_CE
+$Comp
+L power:VCC #PWR0116
+U 1 1 60237F34
+P 2250 3000
+F 0 "#PWR0116" H 2250 2850 50  0001 C CNN
+F 1 "VCC" V 2265 3128 50  0000 L CNN
+F 2 "" H 2250 3000 50  0001 C CNN
+F 3 "" H 2250 3000 50  0001 C CNN
+	1    2250 3000
+	0    1    1    0
+$EndComp
+Wire Wire Line
+	1950 3000 2250 3000
 $EndSCHEMATC
