File: board/pod_27C512/pod_27C512.sch (KiCad schematic (older format))
At the start: 13 parts, among them J1 EXT_D, J2 EXT_ADDR, J3 VCC_Probe, J4 GND_Probe, J5 ROM Lines, U1 74HCT02

Commit message: Force unused address lines to low for 27C512 pod
Connections:
- net A16 is gone; now on net GND: J2.33 (Pin_33)
- net A17 is gone; now on net GND: J2.35 (Pin_35)
- net A18 is gone; now on net GND: J2.37 (Pin_37)
Changed lines of the file:
@@
 Wire Wire Line
 	9950 5600 9550 5600
-Wire Wire Line
-	9950 5700 9550 5700
-Wire Wire Line
-	9950 5800 9550 5800
-Wire Wire Line
-	9950 5900 9550 5900
 Text Label 9550 4100 0    50   ~ 0
 A0
@@
 Wire Wire Line
 	1950 3000 2250 3000
+$Comp
+L power:GND #PWR?
+U 1 1 5FBD02DE
+P 9350 6100
+F 0 "#PWR?" H 9350 5850 50  0001 C CNN
+F 1 "GND" H 9355 5927 50  0000 C CNN
+F 2 "" H 9350 6100 50  0001 C CNN
+F 3 "" H 9350 6100 50  0001 C CNN
+	1    9350 6100
+	1    0    0    -1
+$EndComp
+Wire Wire Line
+	9350 5700 9350 5800
+Wire Wire Line
+	9350 5700 9950 5700
+Wire Wire Line
+	9350 5800 9950 5800
+Connection ~ 9350 5800
+Wire Wire Line
+	9350 5800 9350 5900
+Wire Wire Line
+	9350 5900 9950 5900
+Connection ~ 9350 5900
+Wire Wire Line
+	9350 5900 9350 6100
 $EndSCHEMATC

Commit message: Update the 27C512 pod by adding a protection diode
Parts:
- added D3: BAT48ZFILM, Diode_SMD:D_SOD-123, symbol Diode:BAT48ZFILM
Connections:
- net EXT_VCC: now also D3.1 (K); no longer J5.2 (Pin_2)
- new net: D3.2 (A), J5.2 (Pin_2)
Changed lines of the file:
@@
 Wire Wire Line
 	5300 1350 5300 1450
-Text Label 4750 1350 0    50   ~ 0
+Text Label 4150 1350 0    50   ~ 0
 EXT_VCC
 $Comp
@@
 	5150 1650 5150 1350
 Connection ~ 5150 1350
-Wire Wire Line
-	5150 1350 4750 1350
 $Comp
 L power:GND #PWR0109
@@
 $EndComp
 Wire Wire Line
-	6800 3100 7200 3100
-Text Label 7200 3100 2    50   ~ 0
+	7500 3100 7900 3100
+Text Label 7900 3100 2    50   ~ 0
 EXT_VCC
 Wire Wire Line
@@
 	1950 3000 2250 3000
 $Comp
-L power:GND #PWR?
+L power:GND #PWR0114
 U 1 1 5FBD02DE
 P 9350 6100
-F 0 "#PWR?" H 9350 5850 50  0001 C CNN
+F 0 "#PWR0114" H 9350 5850 50  0001 C CNN
 F 1 "GND" H 9355 5927 50  0000 C CNN
 F 2 "" H 9350 6100 50  0001 C CNN
@@
 Wire Wire Line
 	9350 5900 9350 6100
+$Comp
+L Diode:BAT48ZFILM D3
+U 1 1 5FD6EBED
+P 7350 3100
+F 0 "D3" H 7350 2883 50  0000 C CNN
+F 1 "BAT48ZFILM" H 7350 2974 50  0000 C CNN
+F 2 "Diode_SMD:D_SOD-123" H 7350 2925 50  0001 C CNN
+F 3 "www.st.com/resource/en/datasheet/bat48.pdf" H 7350 3100 50  0001 C CNN
+	1    7350 3100
+	-1   0    0    1
+$EndComp
+Wire Wire Line
+	4150 1350 5150 1350
+Wire Wire Line
+	6800 3100 7200 3100
 $EndSCHEMATC

Commit message: Update 27C512 pod
Parts:
- removed D1: RED, LED_SMD:LED_1206_3216Metric, symbol Device:LED_Small
- removed R2: 1k, Resistor_SMD:R_1206_3216Metric, symbol Device:R_Small
- added F1: 200mA, Fuse:Fuse_1206_3216Metric, symbol Device:Polyfuse_Small
Connections:
- net VCC: now also R1.2, U1.2, U1.3, F1.2
- removed net EXT_VCC: D3.1 (K), R1.2, U1.2, U1.3
- new net: D3.1 (K), F1.1
Changed lines of the file:
@@
 Title ""
 Date ""
-Rev ""
+Rev "1.1"
 Comp ""
 Comment1 ""
@@
 Wire Wire Line
 	5300 1350 5300 1450
-Text Label 4150 1350 0    50   ~ 0
-EXT_VCC
 $Comp
 L Device:R_Small R1
@@
 Wire Wire Line
 	5150 1650 5150 1350
-Connection ~ 5150 1350
 $Comp
 L power:GND #PWR0109
@@
 	1    0    0    -1
 $EndComp
-Wire Wire Line
-	7500 3100 7900 3100
-Text Label 7900 3100 2    50   ~ 0
-EXT_VCC
 Wire Wire Line
 	6800 3200 7200 3200
@@
 A14
 $Comp
-L Device:LED_Small D1
-U 1 1 601944B8
-P 1550 2550
-F 0 "D1" H 1550 2785 50  0000 C CNN
-F 1 "RED" H 1550 2694 50  0000 C CNN
-F 2 "LED_SMD:LED_1206_3216Metric" V 1550 2550 50  0001 C CNN
-F 3 "~" V 1550 2550 50  0001 C CNN
-	1    1550 2550
-	1    0    0    -1
-$EndComp
-$Comp
-L Device:R_Small R2
-U 1 1 6019F326
-P 1850 2550
-F 0 "R2" V 2046 2550 50  0000 C CNN
-F 1 "1k" V 1955 2550 50  0000 C CNN
-F 2 "Resistor_SMD:R_1206_3216Metric" H 1850 2550 50  0001 C CNN
-F 3 "~" H 1850 2550 50  0001 C CNN
-	1    1850 2550
-	0    -1   -1   0
-$EndComp
-Wire Wire Line
-	1750 2550 1650 2550
-$Comp
-L power:GND #PWR0115
-U 1 1 601B232D
-P 1350 2600
-F 0 "#PWR0115" H 1350 2350 50  0001 C CNN
-F 1 "GND" H 1355 2427 50  0000 C CNN
-F 2 "" H 1350 2600 50  0001 C CNN
-F 3 "" H 1350 2600 50  0001 C CNN
-	1    1350 2600
-	1    0    0    -1
-$EndComp
-Wire Wire Line
-	1450 2550 1350 2550
-Wire Wire Line
-	1350 2550 1350 2600
-Wire Wire Line
-	1950 2550 2400 2550
-Text Label 2400 2550 2    50   ~ 0
-EXT_VCC
-$Comp
 L Device:LED_Small D2
 U 1 1 601DEA89
@@
 $EndComp
 Wire Wire Line
-	4150 1350 5150 1350
-Wire Wire Line
 	6800 3100 7200 3100
+$Comp
+L power:VCC #PWR?
+U 1 1 600CD382
+P 4750 1100
+F 0 "#PWR?" H 4750 950 50  0001 C CNN
+F 1 "VCC" H 4765 1273 50  0000 C CNN
+F 2 "" H 4750 1100 50  0001 C CNN
+F 3 "" H 4750 1100 50  0001 C CNN
+	1    4750 1100
+	1    0    0    -1
+$EndComp
+Wire Wire Line
+	4750 1100 4750 1350
+Wire Wire Line
+	4750 1350 5150 1350
+Connection ~ 5150 1350
+$Comp
+L Device:Polyfuse_Small F1
+U 1 1 600E1A2B
+P 7750 3100
+F 0 "F1" V 7955 3100 50  0000 C CNN
+F 1 "200mA" V 7864 3100 50  0000 C CNN
+F 2 "Fuse:Fuse_1206_3216Metric" H 7800 2900 50  0001 L CNN
+F 3 "~" H 7750 3100 50  0001 C CNN
+	1    7750 3100
+	0    -1   -1   0
+$EndComp
+$Comp
+L power:VCC #PWR?
+U 1 1 6010CD32
+P 8050 2950
+F 0 "#PWR?" H 8050 2800 50  0001 C CNN
+F 1 "VCC" H 8065 3123 50  0000 C CNN
+F 2 "" H 8050 2950 50  0001 C CNN
+F 3 "" H 8050 2950 50  0001 C CNN
+	1    8050 2950
+	1    0    0    -1
+$EndComp
+Wire Wire Line
+	8050 2950 8050 3100
+Wire Wire Line
+	8050 3100 7850 3100
+Wire Wire Line
+	7650 3100 7500 3100
 $EndSCHEMATC
