File: board/EproSim/EproSim.kicad_pcb (KiCad board)
At the start: 2 copper layers, 170.2 x 78.7 mm, 88 parts, among them J1 AVR-ISP-6, J2 RS232, J3 Power IN, J4 EXT_ADDR, J5 EXT_D, J6 External Reset, Q1 2N3904, SW1 SW_Push, SW2 Power, U1 ATmega8A-PU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

Commit message: Rev 1.1 of the board, and initial readme
Parts:
- added J7: External RESET, Connector_PinSocket_2.54mm:PinSocket_1x02_P2.54mm_Vertical, F.Cu at (231.1, 128.3)
- added Q2: 2N3906, Package_TO_SOT_THT:TO-92_Inline, F.Cu at (115.6, 130.8)
- added R28: 10, Resistor_THT:R_Axial_DIN0204_L3.6mm_D1.6mm_P7.62mm_Horizontal, F.Cu at (237.5, 128.3)
- added R29: 10, Resistor_THT:R_Axial_DIN0204_L3.6mm_D1.6mm_P7.62mm_Horizontal, F.Cu at (219.7, 128.3)
- added R30: 10K, Resistor_THT:R_Axial_DIN0204_L3.6mm_D1.6mm_P7.62mm_Horizontal, F.Cu at (100.3, 130.8)
- J4, J5: footprint Connector_IDC:IDC-Header_2x20_P2.54mm_Vertical -> Connector_PinHeader_2.54mm:PinHeader_2x20_P2.54mm_Vertical
- J6: value External Reset -> External ~RESET
- R24: value 1K -> 10K
- SW2: footprint Button_Switch_THT:SW_Slide_1P2T_CK_OS102011MS2Q -> EproSim:Slide_Switch
- moved R24 8.89 mm to (100.3, 128.3)
- moved J6 2.54 mm to (248.9, 128.3), turned to 90 degrees
- moved Q1 1.80 mm to (120.7, 128.3)
Connections:
- Q1 pad 3: /~EXT_RESET -> Net-(Q1-Pad3)
Routing:
- net /~EXT_RESET: track 147.1 -> 19.4 mm
- net Net-(Q1-Pad3): track 0.00 -> 120.6 mm
- net Net-(Q2-Pad1): track 0.00 -> 107.0 mm
- net /SRAM_A5: track 171.6 -> 207.3 mm
- net VCC: track 715.6 -> 737.0 mm
- net /EXT_A2: track 125.9 -> 116.7 mm, vias 0 -> 2
- net Net-(Q1-Pad2): track 5.08 -> 14.0 mm
- net /MCU_RESET: track 7.45 -> 16.2 mm
- net Net-(Q2-Pad2): track 0.00 -> 8.15 mm
- net /EXT_RESET: track 0.00 -> 6.35 mm
- net GND: track 879.2 -> 880.9 mm
- net /EXT_D10: track 98.7 -> 99.4 mm
- net /EXT_D8: track 113.5 -> 114.2 mm
- net /EXT_D9: track 107.0 -> 107.5 mm
Other:
- board text added: "A0"
- board text added: "A1"
- board text added: "A10"
- board text added: "A11"
- board text added: "A12"
- board text added: "A13"
- board text added: "A14"
- board text added: "A15"
- board text added: "A16"
- board text added: "A17"
- board text added: "A18"
- board text added: "A2"
- board text added: "A3"
- board text added: "A4"
- board text added: "A5"
- board text added: "A6"
- board text added: "A7"
- board text added: "A8"
- board text added: "A9"
- board text added: "D0"
- board text added: "D1"
- board text added: "D10"
- board text added: "D11"
- board text added: "D12"
- board text added: "D13"
- board text added: "D14"
- board text added: "D15"
- board text added: "D2"
- board text added: "D3"
- board text added: "D4"
- board text added: "D5"
- board text added: "D6"
- board text added: "D7"
- board text added: "D8"
- board text added: "D9"
- board text added: "GND"
- board text added: "VCC"
- board text added: "rev. 1.1"
- board text added: "~CE"
- board text added: "~OE"
- board text added: "~RESET"
- board text added: "~RST"
- board text removed: "External Reset"
- board text removed: "rev.1"
