File: board/pod_27C400/pod_27C400.kicad_pcb (KiCad board)
At the start: 2 copper layers, 43.2 x 58.4 mm, 13 parts, among them J1 EXT_D, J2 EXT_ADDR, J5 ROM Lines, U1 74HCT02

Commit message: Update all the pods to include the diode
Parts:
- added D3: BAT48ZFILM, Diode_SMD:D_SOD-123, F.Cu at (161.8, 86.9)
- renumbered Vcc to J3, GND to J4, ~OE to JP1
Connections:
- J5 pad 40: /EXT_VCC -> Net-(D3-Pad2)
Routing:
- net Net-(D3-Pad2): track 0.00 -> 7.31 mm
- net /EXT_VCC: track 30.3 -> 25.1 mm

Commit message: Update 27C400 Pod
Parts:
- removed D1: RED, LED_SMD:LED_1206_3216Metric
- removed R2: 1k, Resistor_SMD:R_1206_3216Metric
- added F1: 200mA, Fuse:Fuse_1206_3216Metric, F.Cu at (154.3, 88.9)
- moved D3 1.38 mm to (160.7, 87.6), turned to 0 degrees
Connections:
- D3 pad 1: /EXT_VCC -> Net-(D3-Pad1)
- R1 pad 2: /EXT_VCC -> VCC
- U1 pad 2: /EXT_VCC -> VCC
- U1 pad 3: /EXT_VCC -> VCC
Routing:
- net /EXT_VCC: track 25.1 -> 0.00 mm, vias 1 -> 0
- net VCC: track 69.5 -> 86.4 mm, vias 1 -> 2
- net Net-(D3-Pad1): track 0.00 -> 6.03 mm
- net Net-(D1-Pad2): track 3.80 -> 0.00 mm
- net GND: track 196.0 -> 192.3 mm
- net Net-(D3-Pad2): track 7.31 -> 8.17 mm
Other:
- board text added: "rev 1.1"
